File: eagle/projects/ssc_32u_power_board/ssc_32u_power_board.brd (EAGLE design)
At the start: 89.2 x 69 mm, 14 parts, among them J1 691256610002, J14 MOL-SL-3-RA, J15 ESQ-103-24-H-S, J16 691256610002, J2 4x3_2.54MM_HEADER, J3 4x3_2.54MM_HEADER, J4 4x3_2.54MM_HEADER, J5 4x3_2.54MM_HEADER, J6 4x3_2.54MM_HEADER, J7 4x3_2.54MM_HEADER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

Commit message: Added caps
Parts:
- removed J15: ESQ-103-24-H-S, ssc_32u_power_board:ESQ-103-24-H-S
- added C1, C2: (no value), rcl:E5-13
- added J10: ESQ-104-24-H-S, ssc_32u_power_board:ESQ-104-24-H-S
- moved J14 15.8 mm to (77.8, 31.5), flipped to the bottom, turned to 90 degrees
Connections:
- removed net BBB_RX_SSC_TX: J14.3, J15.3
- new net BBB_TX_SSC_TX: J10.3, J14.2
- net BBB_TX_SSC_RX: now also J10.2, J14.3; no longer J14.2, J15.2
- net GND: now also C1.-, C2.-, J10.1; no longer J15.1
- net VBAT_1_FUSE_0_15: now also C1.+
- net VBAT_2_FUSE_16_24_31: now also C2.+
Routing:
- net VBAT_1_FUSE_0_15: track 111.3 -> 71.9 mm
- net GND: track 145.4 -> 108.7 mm
- net BBB_TX_SSC_TX: track 0.00 -> 21.5 mm
- net BBB_RX_SSC_TX: track 19.6 -> 0.00 mm
- net BBB_TX_SSC_RX: track 19.6 -> 21.9 mm
- added copper zone on layer 15, net BATT_1_VDD
- added copper zone on layer 2, net BATT_1_VDD
- added copper zone on layer 15, net BATT_2_VDD
- added copper zone on layer 2, net BATT_2_VDD
- added copper zone on layer 15, net GND
- added copper zone on layer 2, net GND
- added copper zone on layer 15, net VBAT_1_FUSE_0_15
- added copper zone on layer 2, net VBAT_1_FUSE_0_15
- added copper zone on layer 15, net VBAT_2_FUSE_16_24_31
- added copper zone on layer 2, net VBAT_2_FUSE_16_24_31
Other:
- board size 89.2 x 69 mm -> 83.2 x 69 mm
- board text added: "2017"
- board text added: "MC_TX_SSC_RX"
- board text added: "MC_TX_SSC_TX"
- board text added: "SSC-32U Power Board"
- board text added: "Steven Giewont"
